Commit message: functionallity complete

File: src/my_robot/urdf/my_robot.xacro (robot description, xacro)
@@ -30,4 +30,9 @@
         <box size=".4 .2 .1"/>
       </geometry>
+      <material>
+        <ambient>0.2 0.2 1 1</ambient>
+        <diffuse>0.1 0.1 1 1</diffuse>
+        <emissive>0 0 0 1</emissive>
+      </material>
     </visual>
     <collision name='back_caster_collision'>

Commit message: robot model updated

File: src/my_robot/urdf/my_robot.xacro (robot description, xacro)
@@ -22,5 +22,5 @@
       <origin xyz="0 0 0" rpy=" 0 0 0"/>
       <geometry>
-        <box size=".4 .2 .1"/>
+        <box size=".4 .2 .3"/>
       </geometry>
     </collision>
@@ -28,14 +28,9 @@
       <origin xyz="0 0 0" rpy=" 0 0 0"/>
       <geometry>
-        <box size=".4 .2 .1"/>
+        <box size=".4 .2 .3"/>
       </geometry>
-      <material>
-        <ambient>0.2 0.2 1 1</ambient>
-        <diffuse>0.1 0.1 1 1</diffuse>
-        <emissive>0 0 0 1</emissive>
-      </material>
     </visual>
     <collision name='back_caster_collision'>
-      <origin xyz="-0.15 0 -0.05" rpy=" 0 0 0"/>
+      <origin xyz="-0.15 0 -0.15" rpy=" 0 0 0"/>
       <geometry>
         <sphere radius="0.0499"/>
@@ -43,5 +38,5 @@
     </collision>
     <visual name='back_caster_visual'>
-      <origin xyz="-0.15 0 -0.05" rpy=" 0 0 0"/>
+      <origin xyz="-0.15 0 -0.15" rpy=" 0 0 0"/>
       <geometry>
         <sphere radius="0.05"/>
@@ -49,5 +44,5 @@
     </visual>
     <collision name='front_caster_collision'>
-      <origin xyz="0.15 0 -0.05" rpy=" 0 0 0"/>
+      <origin xyz="0.15 0 -0.15" rpy=" 0 0 0"/>
       <geometry>
         <sphere radius="0.0499"/>
@@ -55,5 +50,5 @@
     </collision>
     <visual name='front_caster_visual'>
-      <origin xyz="0.15 0 -0.05" rpy=" 0 0 0"/>
+      <origin xyz="0.15 0 -0.15" rpy=" 0 0 0"/>
       <geometry>
         <sphere radius="0.05"/>
@@ -65,5 +60,5 @@
       <origin xyz="0 0 0" rpy=" 0 1.5707 1.5707"/>
       <geometry>
-        <cylinder radius="0.1" length="0.05"/>
+        <cylinder radius="0.2" length="0.05"/>
       </geometry>
     </visual>
@@ -71,5 +66,5 @@
       <origin xyz="0 0 0" rpy=" 0 1.5707 1.5707"/>
       <geometry>
-        <cylinder radius="0.1" length="0.05"/>
+        <cylinder radius="0.2" length="0.05"/>
       </geometry>
     </collision>
@@ -92,9 +87,9 @@
     <dynamics damping="1.0" friction="1.0"/>
   </joint>
-    <link name="right_wheel">
+  <link name="right_wheel">
     <visual name='right_wheel_vis'>
       <origin xyz="0 0 0" rpy=" 0 1.5707 1.5707"/>
       <geometry>
-        <cylinder radius="0.1" length="0.05"/>
+        <cylinder radius="0.2" length="0.05"/>
       </geometry>
     </visual>
@@ -102,5 +97,5 @@
       <origin xyz="0 0 0" rpy=" 0 1.5707 1.5707"/>
       <geometry>
-        <cylinder radius="0.1" length="0.05"/>
+        <cylinder radius="0.2" length="0.05"/>
       </geometry>
     </collision>
@@ -176,5 +171,5 @@
   </link>
   <joint type="fixed" name="hokuyo_joint">
-    <origin xyz="0.15 0 0.1" rpy="0 0 0"/>
+    <origin xyz="0.15 0 0.2" rpy="0 0 0"/>
     <child link="hokuyo"/>
     <parent link="chassis"/>
